File: hhkb-7u-spacebar-with-macros (1).kicad_pcb (KiCad board)
At the start: 2 copper layers, 344.1 x 101.2 mm, 155 parts, among them SW1 SW_PUSH, U2 ATMEGA32U4, X2 XTAL_GND

Commit message: Schematic with Footprints and Netlist
This is a pre check in before I attempt to import the new net list and update/add/remove components based on the schematic.
Parts:
- D_, D_0, D_1, D_2, D_3, D_4, D_5, D_6, D_7, D_8, D_9, D_A, D_ALT, D_ALT1, D_B, D_BACKSPACE, D_BSLSH, D_C, D_CAPS_LOCK, D_COMMA, D_D, D_DOT, D_E, D_ENTER, D_EQUAL, D_F, D_F1, D_F10, D_F2, D_F3, D_F4, D_F5, D_F6, D_F7, D_F8, D_F9, D_FN, D_G, D_H, D_I, D_J, D_K, D_L, D_M, D_MINUS, D_N, D_O, D_P, D_Q, D_QUOTE, D_R, D_S, D_SEMIC, D_SHIFT, D_SHIFT1, D_SLASH, D_T, D_TAB, D_U, D_V, D_W, D_WIN, D_WIN1, D_X, D_Y, D_Z, D_[, D_], D_`, D_`1: footprint keyboard_parts:D_SOD123_axial -> keyboard_parts:D_SOD123
- moved R6 21.7 mm to (251.5, 111.8), turned to 90 degrees
- moved C10 7.79 mm to (232.4, 109.0), turned to 180 degrees
- moved R5 3.25 mm to (232.4, 103.4), turned to 180 degrees
- moved C14 2.84 mm to (256.5, 111.8)
- moved C8 2.84 mm to (237.5, 96.5), turned to 90 degrees
- moved C11 2.84 mm to (256.5, 100.3)
- moved C12 2.84 mm to (256.5, 104.1)
- moved C13 2.84 mm to (256.5, 108.0)
- moved C9 2.84 mm to (247.7, 96.5), turned to 90 degrees
- moved U2 2.84 mm to (242.6, 109.2)
- moved X2 2.54 mm to (242.6, 96.5), turned to 90 degrees
