File: pcb-project.kicad_pcb (KiCad board)
At the start: 2 copper layers, 328.6 x 100 mm, 146 parts, among them SW1 SW_PUSH, U2 ATMEGA32U4, X2 XTAL_GND

Commit message: RGB Tracing Completed
Ready for production files to be created and sent off to JLCPCB.
Parts:
- added D_RGB1: WS2812B, LED_SMD:LED_WS2812B_PLCC4_5.0x5.0mm_P3.2mm, F.Cu at (54.8, 112.7)
- added D_RGB2: WS2812B, LED_SMD:LED_WS2812B_PLCC4_5.0x5.0mm_P3.2mm, F.Cu at (54.8, 105.6)
- added D_RGB3: WS2812B, LED_SMD:LED_WS2812B_PLCC4_5.0x5.0mm_P3.2mm, F.Cu at (54.8, 98.4)
- added D_RGB4: WS2812B, LED_SMD:LED_WS2812B_PLCC4_5.0x5.0mm_P3.2mm, F.Cu at (54.8, 91.3)
- added D_RGB5: WS2812B, LED_SMD:LED_WS2812B_PLCC4_5.0x5.0mm_P3.2mm, F.Cu at (54.8, 84.1)
- added D_RGB6: WS2812B, LED_SMD:LED_WS2812B_PLCC4_5.0x5.0mm_P3.2mm, F.Cu at (54.8, 77.0)
- added D_RGB7: WS2812B, LED_SMD:LED_WS2812B_PLCC4_5.0x5.0mm_P3.2mm, F.Cu at (54.8, 69.8)
- added D_RGB8: WS2812B, LED_SMD:LED_WS2812B_PLCC4_5.0x5.0mm_P3.2mm, F.Cu at (54.8, 62.7)
- added R9: 500Ω, Resistor_SMD:R_0805_2012Metric, B.Cu at (53.2, 122.2)
Routing:
- net GND: track 223.2 -> 285.5 mm, vias 4 -> 5
- net +5V: track 169.2 -> 218.8 mm, vias 6 -> 9
- net row2: track 345.6 -> 362.6 mm
- net Net-(R9-Pad2): track 0.00 -> 12.3 mm, vias 0 -> 2
- net rgb: track 0.00 -> 7.46 mm, vias 0 -> 1
- net Net-(D_RGB7-Pad2): track 0.00 -> 4.28 mm
- net Net-(D_RGB6-Pad2): track 0.00 -> 4.28 mm
- net Net-(D_RGB5-Pad2): track 0.00 -> 4.28 mm
- net Net-(D_RGB2-Pad2): track 0.00 -> 4.28 mm
- net Net-(D_RGB1-Pad2): track 0.00 -> 4.28 mm
- net Net-(D_RGB4-Pad2): track 0.00 -> 4.28 mm
- net Net-(D_RGB3-Pad2): track 0.00 -> 4.28 mm
- added copper zone on B.Cu, net GND
Other:
- board text added: "PCB-Project v0.2"
- board text removed: "PCB-Project v0.1"
