File: pcb-project.kicad_pcb (KiCad board)
At the start: 2 copper layers, 328.6 x 100 mm, 155 parts, among them SW1 SW_PUSH, U2 ATMEGA32U4, X2 XTAL_GND

Commit message: Removed Unnecessary Resistor on RGB Data Trace
Parts:
- removed R9: 500Ω, Resistor_SMD:R_0805_2012Metric
Connections:
- U2 pad 12: Net-(R9-Pad2) -> rgb
Routing:
- net rgb: track 7.46 -> 21.6 mm, vias 1 -> 3
- net Net-(R9-Pad2): track 12.3 -> 0.00 mm, vias 2 -> 0
